Commit message: clean version

File: openreal2sim/simulation/isaaclab/assets/franka_fr3/franka_fr3.urdf (robot description, URDF)
Before this commit: robot fr3, 20 links, 19 joints
Links:
- removed link fr3_link0_sc
- removed link fr3_link1_sc
- removed link fr3_link2_sc
- removed link fr3_link3_sc
- removed link fr3_link4_sc
- removed link fr3_link5_sc
- removed link fr3_link6_sc
- removed link fr3_link7_sc
- added link base_link
- added link ee_link
- added link right_gripper, mass 0.01
- link fr3_hand: geometry collision mesh filename=meshes/collision/hand.obj; visual mesh filename=meshes/visual/hand.dae
- link fr3_leftfinger: geometry collision mesh filename=meshes/collision/finger.obj; visual mesh filename=meshes/visual/finger.dae
- link fr3_link0: geometry collision mesh filename=meshes/collision/link0.obj; visual mesh filename=meshes/visual/link0.dae
- link fr3_link1: mass None -> 2.797; geometry collision mesh filename=meshes/collision/link1.obj; visual mesh filename=meshes/visual/link1.dae
- link fr3_link2: mass None -> 2.542; geometry collision mesh filename=meshes/collision/link2.obj; visual mesh filename=meshes/visual/link2.dae
- link fr3_link3: mass None -> 2.2513; geometry collision mesh filename=meshes/collision/link3.obj; visual mesh filename=meshes/visual/link3.dae
- link fr3_link4: mass None -> 2.2037; geometry collision mesh filename=meshes/collision/link4.obj; visual mesh filename=meshes/visual/link4.dae
- link fr3_link5: mass None -> 2.2855; geometry collision mesh filename=meshes/collision/link5.obj; visual mesh filename=meshes/visual/link5.dae
- link fr3_link6: mass None -> 1.353; geometry collision mesh filename=meshes/collision/link6.obj; visual mesh filename=meshes/visual/link6.dae
- link fr3_link7: mass None -> 0.35973; geometry collision mesh filename=meshes/collision/link7.obj; visual mesh filename=meshes/visual/link7.dae
- link fr3_rightfinger: geometry collision mesh filename=meshes/collision/finger.obj; visual mesh filename=meshes/visual/finger.dae
Joints:
- removed joint fr3_link0_sc_joint
- removed joint fr3_link1_sc_joint
- removed joint fr3_link2_sc_joint
- removed joint fr3_link3_sc_joint
- removed joint fr3_link4_sc_joint
- removed joint fr3_link5_sc_joint
- removed joint fr3_link6_sc_joint
- removed joint fr3_link7_sc_joint
- added joint ee_fixed_joint: type fixed, parent fr3_hand, child ee_link, origin xyz=0.0 0. 0.1 rpy=0 0.0 0
- added joint fr3_fixed: type fixed, parent base_link, child fr3_link0, origin xyz=0 0 0.0 rpy=0 0 0.0, axis 0 0 0
- added joint right_gripper: type fixed, parent fr3_link7, child right_gripper, origin xyz=0 0 0.207 rpy=0 0 2.35619449019, axis 0 0 1
- joint fr3_joint1: limit lower=-2.3093 upper=2.3093 effort=87.0 velocity=2.0 -> lower=-2.8973 upper=2.8973 effort=87 velocity=2.1750
- joint fr3_joint2: limit lower=-1.5133 upper=1.5133 effort=87.0 velocity=1.0 -> lower=-1.8326 upper=1.8326 effort=87 velocity=2.1750; origin xyz=0 0 0 rpy=-1.5707963267948966 0 0 -> xyz=0 0 0 rpy=-1.57079632679 0 0
- joint fr3_joint3: limit lower=-2.4937 upper=2.4937 effort=87.0 velocity=1.5 -> lower=-2.8973 upper=2.8973 effort=87 velocity=2.1750; origin xyz=0 -0.316 0 rpy=1.5707963267948966 0 0 -> xyz=0 -0.316 0 rpy=1.57079632679 0 0
- joint fr3_joint4: limit lower=-2.7478 upper=-0.4461 effort=87.0 velocity=1.25 -> lower=-3.0718 upper=-0.1222 effort=87 velocity=2.1750; origin xyz=0.0825 0 0 rpy=1.5707963267948966 0 0 -> xyz=0.0825 0 0 rpy=1.57079632679 0 0
- joint fr3_joint5: limit lower=-2.48 upper=2.48 effort=12.0 velocity=3.0 -> lower=-2.8798 upper=2.8798 effort=12 velocity=2.6100; origin xyz=-0.0825 0.384 0 rpy=-1.5707963267948966 0 0 -> xyz=-0.0825 0.384 0 rpy=-1.57079632679 0 0
- joint fr3_joint6: limit lower=0.8521 upper=4.2094 effort=12.0 velocity=1.5 -> lower=0.4363 upper=4.6251 effort=12 velocity=2.6100; origin xyz=0 0 0 rpy=1.5707963267948966 0 0 -> xyz=0 0 0 rpy=1.57079632679 0 0
- joint fr3_joint7: limit lower=-2.6895 upper=2.6895 effort=12.0 velocity=3.0 -> lower=-3.0543 upper=3.0543 effort=12 velocity=2.6100; origin xyz=0.088 0 0 rpy=1.5707963267948966 0 0 -> xyz=0.088 0 0 rpy=1.57079632679 0 0
- joint fr3_joint8: axis (none) -> 0 0 0
